Commit message: update exercise 3

File: Exercise3/src/fanuc_description/robot/rm-10ia.gazebo.xacro (robot description, xacro)
@@ -187,5 +187,5 @@
         <child link="link6" />
         <axis xyz="0 0 1" />
-        <limit lower="-4.712389" upper="4.712389" effort="0" velocity="0" />
+        <limit lower="-47.12389" upper="47.12389" effort="0" velocity="0" />
     </joint>
     <!--************************************************ flange ********************************************-->

File: Exercise3/src/fanuc_description/robot/rm-10ia.urdf (robot description, URDF)
Before this commit: robot fanuc-rm10ia, 8 links, 7 joints
Joints:
- joint joint6: limit lower=-4.712389 upper=4.712389 effort=0 velocity=0 -> lower=-47.12389 upper=47.12389 effort=0 velocity=0

File: Exercise3/src/fanuc_description/robot/rm-20ia_no_limit.gazebo.xacro (robot description, xacro)
@@ -47,5 +47,5 @@
         <child link="link1" />
         <axis xyz="0 0 1" />
-        <limit lower="0" upper="0" effort="0" velocity="0" />
+        <limit lower="-3.15" upper="3.15" effort="0" velocity="0" />
     </joint>
     <!--************************************************LINK 2********************************************-->
@@ -75,5 +75,5 @@
         <child link="link2" />
         <axis xyz="0 0 1" />
-        <limit lower="0" upper="0" effort="0" velocity="0" />
+        <limit lower="-3.15" upper="3.15" effort="0" velocity="0" />
     </joint>
     <!--************************************************LINK 3********************************************-->
@@ -103,5 +103,5 @@
         <child link="link3" />
         <axis xyz="0 0 1" />
-        <limit lower="0" upper="0" effort="0" velocity="0" />
+        <limit lower="-3.15" upper="3.15" effort="0" velocity="0" />
     </joint>
     <!--************************************************LINK 4********************************************-->
@@ -131,5 +131,5 @@
         <child link="link4" />
         <axis xyz="0 0 1" />
-        <limit lower="0" upper="0" effort="0" velocity="0" />
+        <limit lower="-3.15" upper="3.15" effort="0" velocity="0" />
     </joint>
     <!--************************************************LINK 5********************************************-->
@@ -159,5 +159,5 @@
         <child link="link5" />
         <axis xyz="0 0 1" />
-        <limit lower="0" upper="0" effort="0" velocity="0" />
+        <limit lower="-3.15" upper="3.15" effort="0" velocity="0" />
     </joint>
     <!--************************************************LINK 6********************************************-->
@@ -187,5 +187,5 @@
         <child link="link6" />
         <axis xyz="0 0 1" />
-        <limit lower="0" upper="0" effort="0" velocity="0" />
+        <limit lower="-3.15" upper="3.15" effort="0" velocity="0" />
     </joint>
     <!--************************************************ flange ********************************************-->

File: Exercise3/src/fanuc_description/robot/rm-20ia_no_limit.urdf (robot description, URDF)
Before this commit: robot fanuc-rm20ia, 8 links, 7 joints
Joints:
- joint joint1: limit lower=0 upper=0 effort=0 velocity=0 -> lower=-3.15 upper=3.15 effort=0 velocity=0
- joint joint2: limit lower=0 upper=0 effort=0 velocity=0 -> lower=-3.15 upper=3.15 effort=0 velocity=0
- joint joint3: limit lower=0 upper=0 effort=0 velocity=0 -> lower=-3.15 upper=3.15 effort=0 velocity=0
- joint joint4: limit lower=0 upper=0 effort=0 velocity=0 -> lower=-3.15 upper=3.15 effort=0 velocity=0
- joint joint5: limit lower=0 upper=0 effort=0 velocity=0 -> lower=-3.15 upper=3.15 effort=0 velocity=0
- joint joint6: limit lower=0 upper=0 effort=0 velocity=0 -> lower=-3.15 upper=3.15 effort=0 velocity=0
